File: lx_serial/lx_serial.sch (KiCad schematic (older format))
At the start: 23 parts, among them J1 200LX_02X05, P1 USB_OTG, U1 FT231XS, U2 TRS3243E

Commit message: disconnect shield from gnd in usb serial module
Parts:
- added R5: 0R, Resistors_SMD:R_0805_HandSoldering, symbol R
Connections:
- net GND: now also R5.1; no longer P1.6 (shield)
- new net: P1.6 (shield), R5.2
Changed lines of the file:
@@
 $EndComp
 $Comp
-L GND #PWR2
+L GND #PWR01
 U 1 1 577D5483
 P 4500 3850
-F 0 "#PWR2" H 4500 3600 50  0001 C CNN
+F 0 "#PWR01" H 4500 3600 50  0001 C CNN
 F 1 "GND" H 4505 3677 50  0000 C CNN
 F 2 "" H 4500 3850 50  0000 C CNN
@@
 $EndComp
 $Comp
-L AB2_5VUSB #PWR1
+L AB2_5VUSB #PWR02
 U 1 1 577D551A
 P 3450 1200
-F 0 "#PWR1" H 3450 1500 60  0001 C CNN
+F 0 "#PWR02" H 3450 1500 60  0001 C CNN
 F 1 "AB2_5VUSB" H 3450 1400 60  0001 C CNN
 F 2 "" H 3450 1200 60  0000 C CNN
@@
 Connection ~ 3850 3200
 Wire Wire Line
-	2850 3100 2850 3200
+	2850 3200 2850 3100
 Connection ~ 2850 3200
 Wire Wire Line
-	3150 3100 3150 3200
+	3150 3200 3150 3100
 Connection ~ 3150 3200
 Wire Wire Line
-	3450 3100 3450 3200
+	3450 3200 3450 3100
 Connection ~ 3450 3200
 Connection ~ 2650 3200
@@
 	3000 1500 3000 1350
 Connection ~ 3000 1350
-Wire Wire Line
-	2200 3200 3850 3200
 Wire Wire Line
 	6450 1400 6450 1350
@@
 Text Label 2800 2450 0    60   ~ 0
 VUSB_R
+$Comp
+L R R5
+U 1 1 5A89930F
+P 2400 3200
+F 0 "R5" V 2480 3200 50  0000 C CNN
+F 1 "0R" V 2400 3200 50  0000 C CNN
+F 2 "Resistors_SMD:R_0805_HandSoldering" V 2330 3200 50  0001 C CNN
+F 3 "" H 2400 3200 50  0001 C CNN
+	1    2400 3200
+	0    1    1    0
+$EndComp
+Wire Wire Line
+	2200 3200 2250 3200
+Wire Wire Line
+	2550 3200 3850 3200
 $EndSCHEMATC
